File: v1/HWDesign/EAGLE/bluz_gw_v1.brd (EAGLE design)
At the start: 27.9 x 53.3 mm, 29 parts, among them Q1 FC-12M, U2 MDBT40SMD, U3 WM-N-BM-14, U4 SST25VF010A-33-4I-SAE

Commit message: new design files
Parts:
- moved U$2 16.2 mm to (1.24, 33.3)
- moved C4 1.75 mm to (3.68, 46.6)
- moved R2 1.45 mm to (5.87, 46.6)
Routing:
- net VCC: track 152.6 -> 148.9 mm
- net SPI_SS: track 29.2 -> 27.5 mm
- net GND: vias 18 -> 19
Other:
- outline, holes or cut-outs redrawn
- board text added: "Bluz Gateway v1 rev B"
- board text removed: "Bluz Gateway v1 rev A"
Changed lines of the file:
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@@
 <layer number="43" name="vRestrict" color="2" fill="10" visible="yes" active="yes"/>
 <layer number="44" name="Drills" color="7" fill="1" visible="no" active="yes"/>
-<layer number="45" name="Holes" color="7" fill="1" visible="no" active="yes"/>
+<layer number="45" name="Holes" color="7" fill="1" visible="yes" active="yes"/>
 <layer number="46" name="Milling" color="3" fill="1" visible="no" active="yes"/>
 <layer number="47" name="Measures" color="7" fill="1" visible="no" active="yes"/>
@@
 <text x="18.5674" y="28.2194" size="0.8128" layer="25" rot="SR0">1</text>
 <text x="17.526" y="7.8486" size="0.8128" layer="26" rot="MR0">Bluz Gateway
-v1 rev A</text>
+v1 rev B</text>
 <wire x1="2.54" y1="0" x2="0" y2="35.56" width="0" layer="20"/>
-<wire x1="0" y1="35.56" x2="0" y2="53.34" width="0" layer="20"/>
-<wire x1="0" y1="53.34" x2="27.94" y2="53.34" width="0" layer="20"/>
-<wire x1="27.94" y1="53.34" x2="27.94" y2="35.56" width="0" layer="20"/>
+<wire x1="0" y1="35.56" x2="0" y2="45.72" width="0" layer="20"/>
+<wire x1="0" y1="45.72" x2="7.62" y2="53.34" width="0" layer="20"/>
+<wire x1="7.62" y1="53.34" x2="20.32" y2="53.34" width="0" layer="20"/>
+<wire x1="20.32" y1="53.34" x2="27.94" y2="45.72" width="0" layer="20"/>
+<wire x1="27.94" y1="45.72" x2="27.94" y2="35.56" width="0" layer="20"/>
 <wire x1="27.94" y1="35.56" x2="25.4" y2="0" width="0" layer="20"/>
 <wire x1="25.4" y1="0" x2="2.54" y2="0" width="0" layer="20"/>
@@
 <element name="U1" library="Spark" package="SOT223" value="" x="14.224" y="48.895" rot="MR0"/>
 <element name="C3" library="SparkFun-Capacitors" package="0603-CAP" value="0.1uF" x="8.89" y="43.18" rot="MR270"/>
-<element name="U$2" library="bluze_libr" package="BLUZE_LOGO_LOW_RES" value="" x="0.254" y="49.403"/>
+<element name="U$2" library="bluze_libr" package="BLUZE_LOGO_LOW_RES" value="" x="1.2446" y="33.274"/>
 <element name="C2" library="SparkFun-Capacitors" package="0603-CAP" value=".1uF" x="8.89" y="46.99" rot="MR90"/>
 <element name="C7" library="SparkFun-Capacitors" package="0603-CAP" value="1uF" x="20.32" y="43.18" rot="MR90"/>
-<element name="C4" library="SparkFun-Capacitors" package="0603-CAP" value=".1uF" x="2.6924" y="48.0822" rot="R90"/>
-<element name="R2" library="SparkFun-Passives" package="0603-RES" value="1k" x="5.4864" y="48.0314" rot="R270"/>
+<element name="C4" library="SparkFun-Capacitors" package="0603-CAP" value=".1uF" x="3.683" y="46.6344" rot="R90"/>
+<element name="R2" library="SparkFun-Passives" package="0603-RES" value="1k" x="5.8674" y="46.6344" rot="R270"/>
 <element name="FRAME1" library="SparkFun-Aesthetics" package="CREATIVE_COMMONS" value="FRAME-LETTER" x="67.31" y="29.21"/>
 <element name="JP2" library="Spark2" package="USB-A-SMT-MALE" value="USBA-SMD-MALE" x="13.97" y="51.5366" smashed="yes"/>
@@
 <contactref element="C11" pad="2"/>
 <polygon width="0.4064" layer="16">
-<vertex x="0" y="53.34"/>
+<vertex x="-1.27" y="53.34"/>
 <vertex x="0" y="11.43"/>
 <vertex x="23.495" y="11.43"/>
@@
 <via x="5.08" y="31.115" extent="1-16" drill="2.032" shape="octagon"/>
 <via x="22.86" y="31.115" extent="1-16" drill="2.032" shape="octagon"/>
-<via x="3.175" y="51.435" extent="1-16" drill="0.381"/>
-<via x="22.225" y="51.435" extent="1-16" drill="0.381"/>
+<via x="5.9436" y="49.7078" extent="1-16" drill="0.381"/>
+<via x="22.225" y="48.895" extent="1-16" drill="0.381"/>
 <via x="12.065" y="38.735" extent="1-16" drill="0.381"/>
 <wire x1="10.05" y1="35.6526" x2="11.0146" y2="35.6526" width="0.381" layer="1"/>
@@
 <wire x1="11.0654" y1="35.7288" x2="12.1666" y2="36.9316" width="0.254" layer="1"/>
 <contactref element="U4" pad="4"/>
+<via x="1.651" y="45.1104" extent="1-16" drill="0.381"/>
 </signal>
 <signal name="VCC">
@@
 <via x="7.5946" y="45.5676" extent="1-16" drill="0.5588"/>
 <wire x1="8.89" y1="45.5676" x2="7.5946" y2="45.5676" width="0.5588" layer="16"/>
-<wire x1="2.9092" y1="47.0154" x2="2.6924" y2="47.2322" width="0.5588" layer="1"/>
 <wire x1="8.89" y1="46.14" x2="8.89" y2="45.5676" width="0.5588" layer="16"/>
-<wire x1="7.5946" y1="45.5676" x2="7.5946" y2="47.7774" width="0.5588" layer="1"/>
-<wire x1="7.5946" y1="47.7774" x2="6.5532" y2="48.8188" width="0.5588" layer="1"/>
-<wire x1="6.5532" y1="48.8188" x2="4.9784" y2="48.8188" width="0.5588" layer="1"/>
-<wire x1="4.9784" y1="48.8188" x2="3.4036" y2="47.244" width="0.5588" layer="1"/>
-<wire x1="3.4036" y1="47.244" x2="2.7042" y2="47.244" width="0.5588" layer="1"/>
-<wire x1="2.7042" y1="47.244" x2="2.6924" y2="47.2322" width="0.5588" layer="1"/>
-<wire x1="2.9092" y1="47.0154" x2="2.9092" y2="46.4684" width="0.5588" layer="1"/>
-<wire x1="2.9092" y1="46.4684" x2="3.4798" y2="45.8978" width="0.5588" layer="1"/>
-<wire x1="10.05" y1="43.3526" x2="8.89" y2="43.3526" width="0.5588" layer="1"/>
-<wire x1="8.89" y1="43.3526" x2="8.7174" y2="43.3526" width="0.5588" layer="1"/>
+<wire x1="10.05" y1="43.3526" x2="8.7174" y2="43.3526" width="0.5588" layer="1"/>
+<wire x1="8.7122" y1="43.3526" x2="8.7174" y2="43.3526" width="0.5588" layer="1"/>
 <wire x1="8.7174" y1="43.3526" x2="7.62" y2="44.45" width="0.5588" layer="1"/>
 <wire x1="7.62" y1="44.45" x2="7.62" y2="45.5422" width="0.5588" layer="1"/>
 <wire x1="7.62" y1="45.5422" x2="7.5946" y2="45.5676" width="0.5588" layer="1"/>
-<wire x1="7.2898" y1="40.4824" x2="8.89" y2="43.3526" width="0.5588" layer="1"/>
+<wire x1="7.2898" y1="40.4824" x2="8.7122" y2="43.3526" width="0.5588" layer="1"/>
 <wire x1="4.7498" y1="35.3822" x2="2.5654" y2="33.9598" width="0.5588" layer="1"/>
 <wire x1="8.89" y1="44.03" x2="8.89" y2="45.5676" width="0.5588" layer="16"/>
@@
 <wire x1="5.1054" y1="38.227" x2="7.0664" y2="38.227" width="0.5588" layer="1"/>
 <wire x1="7.0664" y1="38.227" x2="7.2898" y2="38.4504" width="0.254" layer="1"/>
-<wire x1="2.5654" y1="43.1546" x2="2.5654" y2="44.9834" width="0.5588" layer="1"/>
-<wire x1="2.5654" y1="44.9834" x2="3.4798" y2="45.8978" width="0.5588" layer="1"/>
+<wire x1="2.6924" y1="43.2816" x2="2.5654" y2="43.1546" width="0.254" layer="1"/>
+<wire x1="2.6924" y1="43.2816" x2="2.6924" y2="44.7938" width="0.254" layer="1"/>
+<wire x1="2.6924" y1="44.7938" x2="3.683" y2="45.7844" width="0.254" layer="1"/>
+<wire x1="3.683" y1="45.7844" x2="4.1674" y2="45.7844" width="0.254" layer="1"/>
+<wire x1="4.1674" y1="45.7844" x2="5.8674" y2="47.4844" width="0.254" layer="1"/>
+<wire x1="5.8674" y1="47.4844" x2="7.1256" y2="47.4844" width="0.254" layer="1"/>
+<wire x1="7.1256" y1="47.4844" x2="7.62" y2="46.99" width="0.254" layer="1"/>
+<wire x1="7.62" y1="46.99" x2="7.62" y2="45.593" width="0.254" layer="1"/>
+<wire x1="7.62" y1="45.593" x2="7.5946" y2="45.5676" width="0.254" layer="1"/>
 <wire x1="18.161" y1="44.7294" x2="18.15" y2="44.8526" width="0" layer="19" extent="1-1"/>
 <wire x1="10.05" y1="43.3526" x2="10.0584" y2="43.3324" width="0" layer="19" extent="1-1"/>
-<wire x1="5.4864" y1="48.8814" x2="4.9784" y2="48.8188" width="0" layer="19" extent="1-1"/>
 </signal>
 <signal name="N$7">
@@
 <wire x1="8.2296" y1="41.3258" x2="5.1308" y2="41.529" width="0.254" layer="16"/>
 <via x="5.1308" y="41.529" extent="1-16" drill="0.3048"/>
-<wire x1="6.0198" y1="46.648" x2="5.4864" y2="47.1814" width="0.5588" layer="1"/>
 <contactref element="U4" pad="1"/>
 <wire x1="5.1308" y1="41.529" x2="5.1308" y2="43.1292" width="0.254" layer="1"/>
 <wire x1="5.1308" y1="43.1292" x2="5.1054" y2="43.1546" width="0.254" layer="1"/>
-<wire x1="5.1054" y1="43.1546" x2="5.1054" y2="45.7336" width="0.5588" layer="1"/>
-<wire x1="5.1054" y1="45.7336" x2="6.0198" y2="46.648" width="0.5588" layer="1"/>
+<wire x1="5.8674" y1="45.7844" x2="5.8674" y2="43.9166" width="0.254" layer="1"/>
+<wire x1="5.8674" y1="43.9166" x2="5.1054" y2="43.1546" width="0.254" layer="1"/>
 </signal>
 <signal name="SPI_MISO">
@@
 <wire x1="4.8514" y1="36.068" x2="5.9436" y2="36.4744" width="0.254" layer="16"/>
 <wire x1="5.9436" y1="36.4744" x2="18.9484" y2="36.4744" width="0.254" layer="16"/>
-<wire x1="18.9484" y1="36.4744" x2="19.5326" y2="36.4236" width="0.254" layer="16"/>
-<via x="19.5326" y="36.4236" extent="1-16" drill="0.3048"/>
-<wire x1="19.5326" y1="36.4236" x2="19.5834" y2="36.2458" width="0.254" layer="1"/>
+<wire x1="18.9484" y1="36.4744" x2="19.558" y2="36.4236" width="0.254" layer="16"/>
+<via x="19.558" y="36.4236" extent="1-16" drill="0.3048"/>
+<wire x1="19.558" y1="36.4236" x2="19.5834" y2="36.2458" width="0.254" layer="1"/>
 <wire x1="19.5834" y1="36.2458" x2="19.5326" y2="35.814" width="0.254" layer="1"/>
 <wire x1="19.5326" y1="35.814" x2="19.5326" y2="34.87" width="0.254" layer="1"/>

Commit message: updated hw design files
Parts:
- added LED2: (no value), led:CHIP-LED0603
- added R5: 1k, SparkFun-Passives:0603-RES
- added R6, R7: 22, SparkFun-Passives:0603-RES
- added S1: (no value), Spark:TACTILE_SWITCH_SMD
- moved C2 0.87 mm to (9.75, 47.1)
- moved C14 0.59 mm to (20.1, 14.5)
- moved C12 0.56 mm to (20.0, 20.6)
- moved C13 0.56 mm to (20.0, 23.7)
- moved C15 0.56 mm to (20.0, 17.6)
- moved C1 0.42 mm to (18.7, 47.2)
Connections:
- new net D7: R5.2, U2.17
- new net MCU_USB_DM: R6.2, U3.62
- new net MCU_USB_DP: R7.2, U3.61
- new net N$5: JP2.D-1, R6.1
- new net N$6: JP2.D+1, R7.1
- new net N$9: LED2.A, R5.1
- new net SETUP: S1.3, S1.4, U3.46
- net GND: now also LED2.C, S1.1, S1.2
- net SA: now also U3.50
Routing:
- net SA: track 0.00 -> 32.2 mm, vias 0 -> 2
- net MCU_USB_DM: track 0.00 -> 29.8 mm, vias 0 -> 2
- net MCU_USB_DP: track 0.00 -> 29.1 mm, vias 0 -> 2
- net N$6: track 0.00 -> 23.0 mm, vias 0 -> 2
- net N$5: track 0.00 -> 21.1 mm, vias 0 -> 2
- net D7: track 0.00 -> 9.65 mm, vias 0 -> 2
- net SETUP: track 0.00 -> 6.28 mm, vias 0 -> 1
- net N$9: track 0.00 -> 2.97 mm
- net N$1: track 17.1 -> 16.4 mm
- net VCC: track 148.9 -> 149.6 mm
- added copper zone on layer 2, net N$10
Other:
- board text added: "Bluz Gateway v1 rev E"
- board text removed: "Bluz Gateway v1 rev B"
