File: v1/HWDesign/EAGLE/bluz_gw_v1.sch (EAGLE design)
At the start: 28 parts, among them Q1 FC-12M, U2 MDBT40SMD, U3 WM-N-BM-14, U4 SST25VF010A-33-4I-SAE

Commit message: new design files
Other:
- note added: "B"
- note removed: "A"
Changed lines of the file:
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@@
 <text x="195.58" y="17.78" size="3.81" layer="94">Bluz Gateway</text>
 <text x="190.246" y="1.27" size="2.54" layer="94">September 2, 2015</text>
-<text x="269.24" y="7.112" size="3.81" layer="94">A</text>
+<text x="269.24" y="7.112" size="3.81" layer="94">B</text>
 <text x="220.98" y="45.72" size="3.048" layer="95">SPI Flash</text>
 <text x="99.06" y="187.96" size="3.048" layer="95">RGB LED</text>

Commit message: updated hw design files
Parts:
- added LED2: (no value), led:LEDCHIP-LED0603
- added R5: 1k, SparkFun-Passives:RESISTOR0603-RES
- added R6, R7: 22, SparkFun-Passives:RESISTOR0603-RES
- added S1: (no value), Spark:TAC_SWITCHSMD
Connections:
- new net D7: R5.2, U2.P0.00
- new net MCU_USB_DM: R6.2, U3.MICRO_UART1_CTS/PA11@62
- new net MCU_USB_DP: R7.2, U3.MICRO_UART1_RTS/PA12@61
- new net N$5: JP2.D-, R6.1
- new net N$6: JP2.D+, R7.1
- new net N$9: LED2.A, R5.1
- new net SETUP: S1.3, S1.4, U3.\MICRO_GPIO_8/PC7@46
- net GND: now also LED2.C, S1.1, S1.2
- net SA: now also U3.MICRO_GPIO_14/PC5@50
Other:
- note added: "E"
- note added: "March 7, 2016"
- note added: "Power/USB"
- note removed: "B"
- note removed: "Power"
- note removed: "September 2, 2015"
- moved on the sheet: C10, C11, C12, C13, C14, C15, C8, C9
